Commit message: Initial commit aus dem alten Repo. Zusätzlich wurde Ultraschallsensor auskommentiert

File: src/osr-rover-code/ROS/osr_gazebo/urdf/gazebo.urdf.xacro (robot description, xacro)
@@ -182,9 +182,9 @@
         </sensor>
     </gazebo>
-    <!-- ───────────── Ultraschall Sensor ───────────── -->
+    <!-- ───────────── Ultraschall Sensor ─────────────
     <link name="ultrasonic_1_link">
       <pose>0.09 -0.139 0.595 0 0 0</pose>
     </link>
-    <joint name="ultrasonic_1_joint" type="fixed">
+      <joint name="ultrasonic_1_joint" type="fixed">
       <parent link="front_wheel_joint_left"/>
       <child  link="ultrasonic_1_link"/>
@@ -230,4 +230,4 @@
         </plugin>
       </sensor>
-    </gazebo>
+    </gazebo> -->
 </robot>

Commit message: Sensor ist jetzt beim Linken Reifen zu sehen aber nur in der Gazebo simulation (Der Parent Link war falsch, es wurde ein "Join" benutz aber es hätte ein "Link" sein müssen

File: src/osr-rover-code/ROS/osr_gazebo/urdf/gazebo.urdf.xacro (robot description, xacro)
@@ -1,3 +1,4 @@
 <?xml version="1.0"?>
+<!--	-->
 <robot xmlns:xacro="http://wiki.ros.org/xacro">
   <ros2_control name="GazeboSystem" type="system">
@@ -182,17 +183,18 @@
         </sensor>
     </gazebo>
-    <!-- ───────────── Ultraschall Sensor ─────────────
+    <!-- ───────────── Ultraschall Sensor ───────────── -->
     <link name="ultrasonic_1_link">
       <pose>0.09 -0.139 0.595 0 0 0</pose>
     </link>
       <joint name="ultrasonic_1_joint" type="fixed">
-      <parent link="front_wheel_joint_left"/>
+      <parent link="front_wheel_link_L"/>
+      <origin xyz="0.10 0.01 -0.16" rpy="0 0 0"/>
       <child  link="ultrasonic_1_link"/>
-      <origin xyz="0.09 -0.139 0.595" rpy="0 0 0"/>
+      <!-- <origin xyz="0.09 -0.139 0.595" rpy="0 0 0"/> -->
     </joint>
     <gazebo reference="ultrasonic_1_link">
       <sensor name="ultrasonic_1" type="ray">
         <always_on>true</always_on>
-        <visualize>false</visualize>
+        <visualize>true</visualize>
         <update_rate>5</update_rate>
         <ray>
@@ -230,4 +232,4 @@
         </plugin>
       </sensor>
-    </gazebo> -->
+    </gazebo>
 </robot>

Commit message: neue Ultraschallsensoren hinzugefügt

File: src/osr-rover-code/ROS/osr_gazebo/urdf/gazebo.urdf.xacro (robot description, xacro)
@@ -176,6 +176,5 @@
                 </range>
             </ray>
-            <plugin name="lidar_plugin"
-                filename="libgazebo_ros_ray_sensor.so">
+            <plugin name="lidar_plugin" filename="libgazebo_ros_ray_sensor.so">
                 <output_type>sensor_msgs/PointCloud</output_type>
                 <frame_name>lidar_link</frame_name>
@@ -184,15 +183,29 @@
     </gazebo>
     <!-- ───────────── Ultraschall Sensor ───────────── -->
-    <link name="ultrasonic_1_link">
+    <xacro:property name="PI" value="3.141592653589793"/>
+    <xacro:macro name="ultra_sensor" params="id parent_link xyz:='0 0 0' rpy:='0 0 0'">
+    <link name="ultrasonic_${id}_link">
       <pose>0.09 -0.139 0.595 0 0 0</pose>
+	<visual>
+    		<origin xyz="0 0 0" rpy="0 0 0"/>
+    		<geometry>
+      			<cylinder radius="0.015" length="0.05"/>
+    		</geometry>
+    		<material name="blue"/>
+  	</visual>
+  	<collision>
+    		<origin xyz="0 0 0" rpy="0 0 0"/>
+    		<geometry>
+      			<cylinder radius="0.015" length="0.05"/>
+    		</geometry>
+  	</collision>
     </link>
-      <joint name="ultrasonic_1_joint" type="fixed">
-      <parent link="front_wheel_link_L"/>
-      <origin xyz="0.10 0.01 -0.16" rpy="0 0 0"/>
-      <child  link="ultrasonic_1_link"/>
-      <!-- <origin xyz="0.09 -0.139 0.595" rpy="0 0 0"/> -->
-    </joint>
-    <gazebo reference="ultrasonic_1_link">
-      <sensor name="ultrasonic_1" type="ray">
+      <joint name="ultrasonic_${id}_joint" type="fixed">
+      	<parent link="${parent_link}"/>
+      	<origin xyz="${xyz}" rpy="${rpy}"/>
+      	<child  link="ultrasonic_${id}_link"/>
+      </joint>
+    <gazebo reference="ultrasonic_${id}_link">
+      <sensor name="ultrasonic_${id}" type="ray">
         <always_on>true</always_on>
         <visualize>true</visualize>
@@ -203,6 +216,6 @@
               <samples>5</samples>
               <resolution>1.0</resolution>
-              <min_angle>-0.12</min_angle>
-              <max_angle>0.12</max_angle>
+              <min_angle>-${7.5 * PI / 180}</min_angle>
+              <max_angle>${7.5 * PI / 180}</max_angle>
             </horizontal>
             <vertical>
@@ -215,5 +228,5 @@
           <range>
             <min>0.02</min>
-            <max>1.0</max>
+            <max>4.0</max>
             <resolution>0.01</resolution>
           </range>
@@ -224,12 +237,18 @@
           </noise>
         </ray>
-         <plugin name="ultrasonic_sensor_1" filename="libgazebo_ros_ray_sensor.so">
-          <ros>
-            <remapping>~/out:=ultrasonic_sensor_1</remapping>
-          </ros>
-          <output_type>sensor_msgs/Range</output_type>
-          <radiation_type>ultrasound</radiation_type>
-        </plugin>
+         <plugin name="ultrasonic_sensor_${id}" filename="libgazebo_ros_ray_sensor.so">
+      		<ros>
+        		<remapping>~/out:=/ultrasonic_sensor_${id}</remapping>
+      		</ros>
+      <output_type>sensor_msgs/Range</output_type>
+      <radiation_type>ultrasound</radiation_type>
+      <frame_name>ultrasonic_${id}_link</frame_name>
+    </plugin>
       </sensor>
     </gazebo>
+   </xacro:macro>
+	<xacro:ultra_sensor id="fl" parent_link="front_wheel_link_L" xyz="0.10 0.01 -0.16" rpy="0 0 0"/>
+	<xacro:ultra_sensor id="fr" parent_link="front_wheel_link_R" xyz="0.10 0.01 -0.16" rpy="0 0 0"/>
+	<xacro:ultra_sensor id="rl" parent_link="rear_wheel_link_L" xyz="-0.10 0.01 -0.16" rpy="0 0 ${PI}"/>
+	<xacro:ultra_sensor id="rr" parent_link="rear_wheel_link_R" xyz="-0.10 0.01 -0.16" rpy="0 0 ${PI}"/>
 </robot>

Commit message: Modelle für Ultraschallsensoren & Lidar Sensor hinzugefügt. Ist nun in Rviz und Gazebo visualisiert. Standfuß für Lidar Sensor selbst erstellt, ggf. nachträglich richtiges Modell von HW Gruppe einfügen

File: src/osr-rover-code/ROS/osr_gazebo/urdf/gazebo.urdf.xacro (robot description, xacro)
@@ -139,4 +139,23 @@
     <!-- ───────────── LiDAR Link und Joint ───────────── -->
     <link name="lidar_link">
+        <visual>
+            <origin xyz="-0.13 -0.027 -0.22" rpy="-1.5708 0 0"/>
+            <geometry>
+               <mesh filename="file://$(find osr_gazebo)/meshes/Lidar.stl" scale="0.001 0.001 0.001"/>
+            </geometry>
+        </visual>
+        <!-- Standfuß -->
+        <visual>
+            <origin xyz ="-0.12 0 -0.265" rpy="0 0 0"/>
+            <geometry>
+               <box size="0.01 0.01 0.05"/>
+            </geometry>
+            <material name="silver"/>
+        </visual>
+        <collision>
+            <geometry>
+               <cylinder radius="0.05" length="0.1"/>
+            </geometry>
+        </collision>
         <inertial>
             <origin xyz="0 0 0" rpy="0 0 0" />
@@ -184,14 +203,23 @@
     <!-- ───────────── Ultraschall Sensor ───────────── -->
     <xacro:property name="PI" value="3.141592653589793"/>
-    <xacro:macro name="ultra_sensor" params="id parent_link xyz:='0 0 0' rpy:='0 0 0'">
+    <xacro:macro name="ultra_sensor" params="id parent_link xyz:='0 0 0' rpy:='0 0 0' vis_x:='0.0' vis_y:='0.0' vis_z:='0.0' b_vis_x:='0.0' b_vis_y:='0.0' b_vis_z:='0.0'">
     <link name="ultrasonic_${id}_link">
       <pose>0.09 -0.139 0.595 0 0 0</pose>
-	<visual>
-    		<origin xyz="0 0 0" rpy="0 0 0"/>
+	<visual> <!-- vorderes Teil -->
+                <!-- Hier NUR das Mesh im Link verschieben/rotieren -->
+    		<origin xyz="${vis_x} ${vis_y} ${vis_z}" rpy="1.5708 ${PI} -1.5708"/>
     		<geometry>
-      			<cylinder radius="0.015" length="0.05"/>
+                        <mesh filename="file://$(find osr_gazebo)/meshes/ultrasonic_front_v6.stl" scale="0.0009 0.0009 0.0009"/>
     		</geometry>
     		<material name="blue"/>
   	</visual>
+	<visual> <!-- Hinteres Teil -->
+                <!-- Hier NUR das Mesh im Link verschieben/rotieren -->
+                <origin xyz="${b_vis_x} ${b_vis_y} ${b_vis_z}" rpy="1.5708 ${PI} 1.5708"/>
+                <geometry>
+                        <mesh filename="file://$(find osr_gazebo)/meshes/ultrasonic_back_v4.stl" scale="0.0009 0.0009 0.0009"/>
+                </geometry>
+                <material name="blue"/>
+        </visual>
   	<collision>
     		<origin xyz="0 0 0" rpy="0 0 0"/>
@@ -248,8 +276,8 @@
     </gazebo>
    </xacro:macro>
-	<xacro:ultra_sensor id="fl" parent_link="front_wheel_link_L" xyz="0.01 -0.04 0" rpy="0 0.785398 0"/>
-	<xacro:ultra_sensor id="fr" parent_link="front_wheel_link_R" xyz="0.01 0.04 0" rpy="0 0.785398 0"/>
-	<xacro:ultra_sensor id="rl" parent_link="rear_wheel_link_L" xyz="-0.01 -0.04 0" rpy="0 0.785398 ${PI}"/>
-	<xacro:ultra_sensor id="rr" parent_link="rear_wheel_link_R" xyz="-0.01 0.04 0" rpy="0 0.785398 ${PI}"/>
+	<xacro:ultra_sensor id="fl" parent_link="front_wheel_link_L" xyz="0.01 -0.04 -0.01" rpy="0 0.785398 0" vis_x="0.012" vis_y="-0.01" vis_z="0.006" b_vis_x="0" b_vis_y="0.026" b_vis_z="0"/>
+	<xacro:ultra_sensor id="fr" parent_link="front_wheel_link_R" xyz="0.01 0.04 -0.01" rpy="0 0.785398 0" vis_x="0.012" vis_y="-0.03" vis_z="0.006" b_vis_x="0" b_vis_y="0.006" b_vis_z="0"/>
+	<xacro:ultra_sensor id="rl" parent_link="rear_wheel_link_L" xyz="-0.01 -0.04 -0.01" rpy="0 0.785398 ${PI}" vis_x="0.012" vis_y="-0.03" vis_z="0.006" b_vis_x="0" b_vis_y="0.006" b_vis_z="0"/>
+	<xacro:ultra_sensor id="rr" parent_link="rear_wheel_link_R" xyz="-0.01 0.04 -0.01" rpy="0 0.785398 ${PI}" vis_x="0.012" vis_y="-0.01" vis_z="0.006" b_vis_x="0" b_vis_y="0.026" b_vis_z="0"/>
 </robot>
 <!--

Commit message: Lidar Standfuß in gazebo.urdf.xacro hinzugefügt

File: src/osr-rover-code/ROS/osr_gazebo/urdf/gazebo.urdf.xacro (robot description, xacro)
@@ -140,5 +140,5 @@
     <link name="lidar_link">
         <visual>
-            <origin xyz="-0.13 -0.027 -0.22" rpy="-1.5708 0 0"/>
+            <origin xyz="-0.135 -0.027 -0.215" rpy="-1.5708 0 0"/>
             <geometry>
                <mesh filename="file://$(find osr_gazebo)/meshes/Lidar.stl" scale="0.001 0.001 0.001"/>
@@ -147,9 +147,9 @@
         <!-- Standfuß -->
         <visual>
-            <origin xyz ="-0.12 0 -0.265" rpy="0 0 0"/>
-            <geometry>
-               <box size="0.01 0.01 0.05"/>
-            </geometry>
-            <material name="silver"/>
+          <origin xyz ="-0.157 0 -0.292" rpy="0 0 -1.5708"/>
+          <geometry>
+            <mesh filename="file://$(find osr_gazebo)/meshes/Lidar_Tower.stl" scale="1 1 1"/>
+          </geometry>
+          <material name="silver"/>
         </visual>
         <collision>

Commit message: Feinjustierung der Lidarposition in der gazebo.urdf.xacro

File: src/osr-rover-code/ROS/osr_gazebo/urdf/gazebo.urdf.xacro (robot description, xacro)
@@ -140,5 +140,5 @@
     <link name="lidar_link">
         <visual>
-            <origin xyz="-0.135 -0.027 -0.215" rpy="-1.5708 0 0"/>
+            <origin xyz="-0.149 -0.027 -0.215" rpy="-1.5708 0 0"/>
             <geometry>
                <mesh filename="file://$(find osr_gazebo)/meshes/Lidar.stl" scale="0.001 0.001 0.001"/>
@@ -147,5 +147,5 @@
         <!-- Standfuß -->
         <visual>
-          <origin xyz ="-0.157 0 -0.292" rpy="0 0 -1.5708"/>
+          <origin xyz ="-0.171 0 -0.292" rpy="0 0 -1.5708"/>
           <geometry>
             <mesh filename="file://$(find osr_gazebo)/meshes/Lidar_Tower.stl" scale="1 1 1"/>

Commit message: Glitchen der Hinterräder in Rviz wurde gefixt. Nun werden die Räder in Rviz normal angezeigt und bewegen sich sogar wie gewünscht parallel zu Gazebo mit richtiger Reifenbewegung

File: src/osr-rover-code/ROS/osr_gazebo/urdf/gazebo.urdf.xacro (robot description, xacro)
@@ -110,4 +110,12 @@
       <state_interface name="velocity"/>
       <state_interface name="effort"/>
+    </joint>
+    <joint name="rocker_bogie_joint_L_2">
+      <state_interface name="position"/>
+      <state_interface name="velocity"/>
+    </joint>
+    <joint name="rocker_bogie_joint_R_2">
+      <state_interface name="position"/>
+      <state_interface name="velocity"/>
     </joint>
   </ros2_control>
